Commit message: Add onboard launch file

File: hector_centaur_description/robots/centaur_default.urdf.xacro (robot description, xacro)
@@ -113,3 +113,75 @@
   </gazebo>
 <!--</macro>-->
+    <xacro:include filename="$(find hector_components_description)/urdf/vision_box_common_dimensions.urdf.xacro" />
+    <xacro:include filename="$(find hector_components_description)/urdf/vision_box_dimensions_hector2.urdf.xacro" />
+    <xacro:include filename="$(find hector_sensors_description)/urdf/hokuyo_utm30lx.urdf.xacro" />
+    <joint name="laser1/x" type="revolute">
+      <origin xyz="${x_vision_box_front} 0 ${laser1RollServo_height}" rpy="0 0 0"/>
+      <parent link="base_link"/>
+      <child link="laser1RollServo"/>
+      <axis xyz="1 0 0"/>
+      <limit lower="${-M_PI/2}" upper="${M_PI/2}" effort="100" velocity="100"/>
+    </joint>
+    <link name="laser1RollServo">
+      <inertial_sphere mass="0.1" diameter="0.07"/>
+      <visual>
+        <origin xyz="${laser1RollServo_size_x/2} 0.0 0.0" rpy="0 0 0"/>
+        <geometry>
+          <box size="${laser1RollServo_size_x} ${laser1RollServo_size_y} ${laser1RollServo_size_z}"/>
+        </geometry>
+        <material name="Blue"/>
+      </visual>
+      <collision>
+        <origin xyz="${laser1RollServo_size_x/2} 0.0 0.0" rpy="0 0 0"/>
+        <geometry>
+          <box size="${laser1RollServo_size_x} ${laser1RollServo_size_y} ${laser1RollServo_size_z}"/>
+        </geometry>
+      </collision>
+    </link>
+    <joint name="laser1/y" type="revolute">
+      <origin xyz="${laser1RollServo_size_x} 0 0" rpy="0 0 0"/>
+      <parent link="laser1RollServo"/>
+      <child link="laser1_link"/>
+      <axis xyz="0 1 0"/>
+      <limit lower="${-M_PI/2}" upper="${M_PI/2}" effort="100" velocity="100"/>
+    </joint>
+    <link name="laser1_link">
+      <inertial_sphere mass="0.1" diameter="0.07"/>
+      <visual>
+        <origin xyz="0.0 0.0 ${laser1_size_z/2}" rpy="0 0 0"/>
+        <geometry>
+          <!--<box size="${laser1_size_x} ${laser1_size_y} ${laser1_size_z}" />-->
+          <box size="${laser1_size_x} ${laser1_size_y} 0.01"/>
+        </geometry>
+        <material name="Grey"/>
+      </visual>
+      <collision>
+        <origin xyz="0.0 0.0 ${laser1_size_z/2}" rpy="0 0 0"/>
+        <geometry>
+          <!--<box size="${laser1_size_x} ${laser1_size_y} ${laser1_size_z}" />-->
+          <box size="${laser1_size_x} ${laser1_size_y} 0.01"/>
+        </geometry>
+      </collision>
+    </link>
+    <xacro:hokuyo_utm30lx name="laser1" parent="laser1_link" ros_topic="laser1/scan" update_rate="40" ray_count="1081" min_angle="-135" max_angle="135">
+      <origin xyz="${laser1_center_x_offset} 0 ${laser1_plane_height}" rpy="0 0 0"/>
+    </xacro:hokuyo_utm30lx>
+    <gazebo>
+      <plugin name="laser1_servo_controller" filename="libhector_servo_plugin.so">
+        <alwaysOn>true</alwaysOn>
+        <controlRate>50.0</controlRate>
+        <updateRate>0.0</updateRate>
+        <firstServoName>laser1/x</firstServoName>
+        <firstServoAxis>1 0 0</firstServoAxis>
+        <secondServoName>laser1/y</secondServoName>
+        <secondServoAxis>0 1 0</secondServoAxis>
+        <torque>0.5</torque>
+        <robotNamespace>/</robotNamespace>
+        <topicName>laser1/command</topicName>
+        <jointStateName>joint_states</jointStateName>
+        <proportionalControllerGain>8.0</proportionalControllerGain>
+        <derivativeControllerGain>0.0</derivativeControllerGain>
+        <maxVelocity>0.0</maxVelocity>
+      </plugin>
+    </gazebo>
 </robot>

Commit message: Add sensor head

File: hector_centaur_description/robots/centaur_default.urdf.xacro (robot description, xacro)
@@ -117,5 +117,5 @@
     <xacro:include filename="$(find hector_sensors_description)/urdf/hokuyo_utm30lx.urdf.xacro" />
     <joint name="laser1/x" type="revolute">
-      <origin xyz="${x_vision_box_front} 0 ${laser1RollServo_height}" rpy="0 0 0"/>
+      <origin xyz="${x_vision_box_front} 0 0.2" rpy="0 0 0"/>
       <parent link="base_link"/>
       <child link="laser1RollServo"/>
@@ -185,3 +185,123 @@
       </plugin>
     </gazebo>
+    <joint name="camera/z" type="revolute">
+      <origin xyz="0.2 0 0.24" rpy="0 0 0"/>
+      <parent link="base_link"/>
+      <child link="cameraYawServo"/>
+      <axis xyz="0 0 1"/>
+      <limit lower="${-M_PI*3/4}" upper="${M_PI*3/4}" effort="100" velocity="100"/>
+    </joint>
+    <link name="cameraYawServo">
+      <inertial_sphere mass="0.1" diameter="0.07"/>
+      <visual>
+        <origin xyz="0.0 0.0 ${cameraYawServo_size_z/2}" rpy="0 0 0"/>
+        <geometry>
+          <box size="${cameraYawServo_size_x} ${cameraYawServo_size_y} ${cameraYawServo_size_z}"/>
+        </geometry>
+        <material name="Blue"/>
+      </visual>
+      <collision>
+        <origin xyz="0.0 0.0 ${cameraYawServo_size_z/2}" rpy="0 0 0"/>
+        <geometry>
+          <box size="${cameraYawServo_size_x} ${cameraYawServo_size_y} ${cameraYawServo_size_z}"/>
+        </geometry>
+      </collision>
+    </link>
+    <joint name="camera/y" type="revolute">
+      <origin xyz="0 0 ${cameraYawServo_size_z}" rpy="0 0 0"/>
+      <parent link="cameraYawServo"/>
+      <child link="mounting_link"/>
+      <axis xyz="0 1 0"/>
+      <limit lower="${-M_PI/2}" upper="${M_PI/2}" effort="100" velocity="100"/>
+    </joint>
+    <link name="mounting_link">
+      <inertial_sphere mass="0.05" diameter="0.07"/>
+    </link>
+    <xacro:include filename="$(find hector_sensors_description)/urdf/thermaleye_camera.urdf.xacro"/>
+    <xacro:thermaleye_camera_model name="infrared" parent="mounting_link">
+      <origin xyz="${infrared_x_position} ${infrared_y_position} ${infrared_z_position}" rpy="0 0 0"/>
+    </xacro:thermaleye_camera_model>
+    <xacro:asus_camera_model name="openni" parent="mounting_link">
+      <origin xyz="${kinect_x_position} ${kinect_y_position}  ${kinect_z_position}" rpy="${kinect_roll_position} ${kinect_pitch_position} ${kinect_yaw_position}"/>
+    </xacro:asus_camera_model>
+    <gazebo>
+      <plugin name="camera_servo_controller" filename="libhector_servo_plugin.so">
+        <alwaysOn>true</alwaysOn>
+        <controlRate>50.0</controlRate>
+        <updateRate>0.0</updateRate>
+        <firstServoName>camera/z</firstServoName>
+        <firstServoAxis>0 0 1</firstServoAxis>
+        <secondServoName>camera/y</secondServoName>
+        <secondServoAxis>0 1 0</secondServoAxis>
+        <torque>0.5</torque>
+        <robotNamespace>/</robotNamespace>
+        <topicName>camera/command</topicName>
+        <jointStateName>joint_states</jointStateName>
+        <proportionalControllerGain>8.0</proportionalControllerGain>
+        <derivativeControllerGain>0.0</derivativeControllerGain>
+        <maxVelocity>2.0</maxVelocity>
+      </plugin>
+    </gazebo>
+    <gazebo reference="openni_depth_frame">
+      <sensor type="depth" name="kinect_camera">
+        <update_rate>10</update_rate>
+        <camera>
+          <horizontal_fov>${60.0*M_PI/180.0}</horizontal_fov>
+          <image>
+            <format>R8G8B8</format>
+            <width>320</width>
+            <height>240</height>
+          </image>
+          <clip>
+            <near>0.05</near>
+            <far>3</far>
+          </clip>
+        </camera>
+        <plugin name="kinect_camera_controller" filename="libgazebo_ros_openni_kinect.so">
+          <alwaysOn>true</alwaysOn>
+          <updateRate>10</updateRate>
+          <imageTopicName>openni/rgb/image_color</imageTopicName>
+          <cameraInfoTopicName>openni/camera_info</cameraInfoTopicName>
+          <depthImageTopicName>openni/depth/image_raw</depthImageTopicName>
+          <depthImageCameraInfoTopicName>openni/depth/camera_info</depthImageCameraInfoTopicName>
+          <pointCloudTopicName>openni/depth/points</pointCloudTopicName>
+          <frameName>openni_depth_optical_frame</frameName>
+          <pointCloudCutoff>0.5</pointCloudCutoff>
+          <distortionK1>0</distortionK1>
+          <distortionK2>0</distortionK2>
+          <distortionK3>0</distortionK3>
+          <distortionT1>0</distortionT1>
+          <distortionT2>0</distortionT2>
+          <CxPrime>0</CxPrime>
+          <Cx>0</Cx>
+          <Cy>0</Cy>
+          <focalLength>0</focalLength>
+          <hackBaseline>0</hackBaseline>
+        </plugin>
+      </sensor>
+    </gazebo>
+    <gazebo reference="infrared_frame">
+      <sensor type="camera" name="thermal_camera_sensor">
+        <update_rate>10</update_rate>
+        <camera>
+          <horizontal_fov>${90.0*M_PI/180.0}</horizontal_fov>
+          <image>
+            <format>R8G8B8</format>
+            <width>160</width>
+            <height>120</height>
+          </image>
+          <clip>
+            <near>0.01</near>
+            <far>100</far>
+          </clip>
+        </camera>
+        <plugin name="thermal_camera_controller" filename="libgazebo_ros_thermal_camera.so">
+          <alwaysOn>true</alwaysOn>
+          <updateRate>10</updateRate>
+          <imageTopicName>/thermal/image</imageTopicName>
+          <cameraInfoTopicName>/thermal/camera_info</cameraInfoTopicName>
+          <frameName>infrared_optical_frame</frameName>
+        </plugin>
+      </sensor>
+    </gazebo>
 </robot>
